File: KiCAD/SmallyMouse2.kicad_sch (KiCad schematic)
At the start: 34 parts, among them IC1 AT90USB1287, J1 Exp Header, J2 Slow/Fast, J3 BBC_UP_02X10, J4 Universal output, J5 Bootloader, J6 Reset, P1 USB_A, Y1 16 MHz Crystal

Commit message: Sync PCB with schematic and finish test-point/junction cleanup
Run Update PCB from Schematic in KiCad 10 so the board carries the
schematic's net names (KiCad 4 auto-names such as Net-(IC1-Pad20)
become Net-(IC1-~{RESET})) plus the pin function/type, sheet and unit
metadata KiCad now stores per footprint. Schematic parity is clean.

- J3 pins 1/19: split the crossing wires at the junctions so the
  editor keeps them (a bare junction on unbroken wires is discarded on
  load); +5V/GND now reach the pads from the schematic side as well
- Test points: KiCad requires numbered references, so return to
  TP1-TP7 in the schematic; on the board hide the reference and show
  the value (RST, TMS, TDI, GND, TCK, TDO, 5V) on the silkscreen at the
  same position, keeping the original silkscreen text
- Test points excluded from BOM and position files on both sides
- KiCad rewrote SmallyMouse2.kicad_pro with its full default set
- Ignore KiCad 10's .history/ local-history directory

Co-Authored-By: Claude Opus 5 <noreply@anthropic.com>
Parts:
- TP1: renamed from RST; value ~{RESET} -> RST
- TP7: renamed from 5V; value +5V -> 5V
- renumbered TMS to TP2, TDI to TP3, GND to TP4, TCK to TP5, TDO to TP6
Changed lines of the file:
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@@
 	(wire
 		(pts
-			(xy 215.9 101.6) (xy 227.33 101.6)
+			(xy 215.9 101.6) (xy 224.79 101.6)
 		)
 		(stroke
@@
 	(wire
 		(pts
-			(xy 224.79 99.06) (xy 224.79 104.14)
+			(xy 224.79 101.6) (xy 227.33 101.6)
+		)
+		(stroke
+			(width 0)
+			(type default)
+		)
+	)
+	(wire
+		(pts
+			(xy 224.79 99.06) (xy 224.79 101.6)
+		)
+		(stroke
+			(width 0)
+			(type default)
+		)
+	)
+	(wire
+		(pts
+			(xy 224.79 101.6) (xy 224.79 104.14)
 		)
 		(stroke
@@
 	(wire
 		(pts
-			(xy 217.17 124.46) (xy 227.33 124.46)
+			(xy 217.17 124.46) (xy 224.79 124.46)
+		)
+		(stroke
+			(width 0)
+			(type default)
+		)
+	)
+	(wire
+		(pts
+			(xy 224.79 124.46) (xy 227.33 124.46)
 		)
 		(stroke
@@
 	(wire
 		(pts
-			(xy 224.79 106.68) (xy 224.79 127)
+			(xy 224.79 106.68) (xy 224.79 124.46)
+		)
+		(stroke
+			(width 0)
+			(type default)
+		)
+	)
+	(wire
+		(pts
+			(xy 224.79 124.46) (xy 224.79 127)
 		)
 		(stroke
@@
 		(in_bom no)
 		(on_board yes)
-		(in_pos_files yes)
+		(in_pos_files no)
 		(dnp no)
-		(property "Reference" "TCK"
+		(property "Reference" "TP5"
 			(at 53.34 106.68 0)
 			(show_name no)
@@
 			(project "SmallyMouse2"
 				(path "/3243e337-5b75-4765-b867-6e38ad1f5f8b"
-					(reference "TCK")
+					(reference "TP5")
 					(unit 1)
 				)
@@
 		(in_bom no)
 		(on_board yes)
-		(in_pos_files yes)
+		(in_pos_files no)
 		(dnp no)
-		(property "Reference" "TMS"
+		(property "Reference" "TP2"
 			(at 45.72 109.22 0)
 			(show_name no)
@@
 			(project "SmallyMouse2"
 				(path "/3243e337-5b75-4765-b867-6e38ad1f5f8b"
-					(reference "TMS")
+					(reference "TP2")
 					(unit 1)
 				)
@@
 		(in_bom no)
 		(on_board yes)
-		(in_pos_files yes)
+		(in_pos_files no)
 		(dnp no)
-		(property "Reference" "TDO"
+		(property "Reference" "TP6"
 			(at 53.34 111.76 0)
 			(show_name no)
@@
 			(project "SmallyMouse2"
 				(path "/3243e337-5b75-4765-b867-6e38ad1f5f8b"
-					(reference "TDO")
+					(reference "TP6")
 					(unit 1)
 				)
@@
 		(in_bom no)
 		(on_board yes)
-		(in_pos_files yes)
+		(in_pos_files no)
 		(dnp no)
-		(property "Reference" "TDI"
+		(property "Reference" "TP3"
 			(at 45.72 114.3 0)
 			(show_name no)
@@
 			(project "SmallyMouse2"
 				(path "/3243e337-5b75-4765-b867-6e38ad1f5f8b"
-					(reference "TDI")
+					(reference "TP3")
 					(unit 1)
 				)
@@
 		(in_bom no)
 		(on_board yes)
-		(in_pos_files yes)
+		(in_pos_files no)
 		(dnp no)
-		(property "Reference" "RST"
+		(property "Reference" "TP1"
 			(at 45.72 102.87 0)
 			(show_name no)
@@
 			)
 		)
-		(property "Value" "~{RESET}"
+		(property "Value" "RST"
 			(at 46.99 102.87 0)
 			(show_name no)
@@
 			(project "SmallyMouse2"
 				(path "/3243e337-5b75-4765-b867-6e38ad1f5f8b"
-					(reference "RST")
+					(reference "TP1")
 					(unit 1)
 				)
@@
 		(in_bom no)
 		(on_board yes)
-		(in_pos_files yes)
+		(in_pos_files no)
 		(dnp no)
-		(property "Reference" "5V"
+		(property "Reference" "TP7"
 			(at 53.34 116.84 0)
 			(show_name no)
@@
 			)
 		)
-		(property "Value" "+5V"
+		(property "Value" "5V"
 			(at 54.61 116.84 0)
 			(show_name no)
@@
 			(project "SmallyMouse2"
 				(path "/3243e337-5b75-4765-b867-6e38ad1f5f8b"
-					(reference "5V")
+					(reference "TP7")
 					(unit 1)
 				)
@@
 		(in_bom no)
 		(on_board yes)
-		(in_pos_files yes)
+		(in_pos_files no)
 		(dnp no)
-		(property "Reference" "GND"
+		(property "Reference" "TP4"
 			(at 45.72 119.38 0)
 			(show_name no)
@@
 			(project "SmallyMouse2"
 				(path "/3243e337-5b75-4765-b867-6e38ad1f5f8b"
-					(reference "GND")
+					(reference "TP4")
 					(unit 1)
 				)
