File: KiCAD/SmallyMouse2.kicad_sch (KiCad schematic)
At the start: 34 parts, among them IC1 AT90USB1287, J1 Exp Header, J2 Slow/Fast, J3 BBC_UP_02X10, J4 Universal output, J5 Bootloader, J6 Reset, P1 USB_A, Y1 16 MHz Crystal

Commit message: Add a note to the schematic about the debug UART Tx and update the schematic page text
Other:
- note added: "Note: PD3 is UART Tx for debug console"
